Commit message: 走路跑步训练更新

File: resources/robots/N2/urdf/N2.urdf (robot description, URDF)
Before this commit: robot N2, 21 links, 20 joints
Links:
- link R_leg_hip_pitch_link: mass 3.1964 -> 3.1965
- link R_leg_knee_link: mass 1.6354 -> 1.6352
Joints:
- joint L_arm_elbow_joint: limit lower=-1.8 upper=1 effort=36 velocity=12 -> lower=-1.8 upper=1 effort=27 velocity=10
- joint L_arm_shoulder_pitch_joint: limit lower=-2.7 upper=2.7 effort=36 velocity=12 -> lower=-2.7 upper=2.7 effort=27 velocity=10
- joint L_arm_shoulder_roll_joint: limit lower=0 upper=2.1 effort=36 velocity=12 -> lower=0 upper=2.1 effort=27 velocity=10
- joint L_arm_shoulder_yaw_joint: limit lower=-2.7 upper=2.7 effort=36 velocity=12 -> lower=-2.7 upper=2.7 effort=27 velocity=10
- joint L_leg_ankle_joint: limit lower=-1 upper=0.75 effort=36 velocity=12 -> lower=-1 upper=0.75 effort=70 velocity=14
- joint R_arm_elbow_joint: limit lower=-1.8 upper=1 effort=36 velocity=12 -> lower=-1.8 upper=1 effort=27 velocity=10; origin xyz=0.0030284 0 -0.17234 rpy=0 0 0 -> xyz=0.0030284 0 -0.17141 rpy=0 0 0
- joint R_arm_hand_joint: origin xyz=-0.0045 0.00018648 -0.18067 rpy=0 0 0 -> xyz=-0.0045 -0.00036368 -0.1815 rpy=0 0 0
- joint R_arm_shoulder_pitch_joint: limit lower=-2.7 upper=2.7 effort=36 velocity=12 -> lower=-2.7 upper=2.7 effort=27 velocity=10
- joint R_arm_shoulder_roll_joint: limit lower=-2.1 upper=0 effort=36 velocity=12 -> lower=-2.1 upper=0 effort=27 velocity=10
- joint R_arm_shoulder_yaw_joint: limit lower=-2.7 upper=2.7 effort=36 velocity=12 -> lower=-2.7 upper=2.7 effort=27 velocity=10
- joint R_leg_ankle_joint: limit lower=-1 upper=0.75 effort=36 velocity=14 -> lower=-1 upper=0.75 effort=70 velocity=14
- joint R_leg_hip_roll_joint: limit lower=-1 upper=0.65 effort=90 velocity=12 -> lower=-1 upper=0.65 effort=90 velocity=14
- joint R_leg_hip_yaw_joint: limit lower=-1 upper=0.65 effort=90 velocity=12 -> lower=-1 upper=0.65 effort=90 velocity=14

File: resources/robots/N2/urdf/N2_10dof.urdf (robot description, URDF)
Before this commit: robot N2, 21 links, 20 joints
Joints:
- joint L_leg_ankle_joint: limit lower=-1 upper=0.75 effort=70 velocity=12 -> lower=-1 upper=0.75 effort=70 velocity=14
- joint L_leg_hip_roll_joint: limit lower=-0.65 upper=1 effort=90 velocity=12 -> lower=-0.65 upper=1 effort=90 velocity=14
- joint L_leg_hip_yaw_joint: limit lower=-0.65 upper=1 effort=90 velocity=12 -> lower=-0.65 upper=1 effort=90 velocity=14
- joint R_arm_elbow_joint: origin xyz=0.0030284 0 -0.17234 rpy=0 0 0 -> xyz=0.0030284 0 -0.17141 rpy=0 0 0
- joint R_arm_hand_joint: origin xyz=-0.0045 0.00018648 -0.18067 rpy=0 0 0 -> xyz=-0.0045 -0.00036368 -0.1815 rpy=0 0 0
- joint R_leg_ankle_joint: limit lower=-1 upper=0.75 effort=70 velocity=12 -> lower=-1 upper=0.75 effort=70 velocity=14
- joint R_leg_hip_roll_joint: limit lower=-1 upper=0.65 effort=90 velocity=12 -> lower=-1 upper=0.65 effort=90 velocity=14
- joint R_leg_hip_yaw_joint: limit lower=-1 upper=0.65 effort=90 velocity=12 -> lower=-1 upper=0.65 effort=90 velocity=14
