Commit message: Initial commit: training framework for N2 humanoid system

File: resources/robots/N2/urdf/N2_10dof.urdf (robot description, URDF)
Before this commit: robot N2, 21 links, 20 joints
Joints:
- joint L_arm_elbow_joint: axis 0 1 0 -> (none); limit lower=-1.8 upper=1 effort=27 velocity=10 -> (none)
- joint L_arm_shoulder_pitch_joint: axis 0 0 1 -> (none); limit lower=-2.7 upper=2.7 effort=27 velocity=10 -> (none)
- joint L_arm_shoulder_roll_joint: limit lower=0 upper=2.1 effort=27 velocity=10 -> (none); origin xyz=0 0 0 rpy=1.5963 0 0 -> xyz=0 0 0 rpy=1.6963 0 0
- joint L_arm_shoulder_yaw_joint: axis 0 0 1 -> (none); limit lower=-2.7 upper=2.7 effort=27 velocity=10 -> (none)
- joint R_arm_elbow_joint: axis 0 1 0 -> (none); limit lower=-1.8 upper=1 effort=27 velocity=10 -> (none)
- joint R_arm_shoulder_pitch_joint: axis 0 0 -1 -> (none); limit lower=-2.7 upper=2.7 effort=27 velocity=10 -> (none)
- joint R_arm_shoulder_roll_joint: limit lower=-2.1 upper=0 effort=27 velocity=10 -> (none); origin xyz=0 0 0 rpy=-1.5963 0 0 -> xyz=0 0 0 rpy=-1.6963 0 0
- joint R_arm_shoulder_yaw_joint: axis 0 0 1 -> (none); limit lower=-2.7 upper=2.7 effort=27 velocity=10 -> (none)
